Commit message: fix o2&cyberdog2 urdf

File: cyberdog2/urdf/cyberdog2.urdf (robot description, URDF)
Before this commit: robot cyberdog2, 40 links, 39 joints
Links:
- link FL_hip_shoulder: geometry collision cylinder length=0.035 radius=0.039; visual cylinder length=0.035 radius=0.039
- link FL_knee: geometry collision box size=0.016 0.016 0.18341; visual mesh filename=package://cyberdog2/meshes/visual/knee.stl scale=1 1 1
- link FR_hip_shoulder: geometry collision cylinder length=0.035 radius=0.039; visual cylinder length=0.035 radius=0.039
- link FR_knee: geometry collision box size=0.016 0.016 0.18341; visual mesh filename=package://cyberdog2/meshes/visual/knee.stl scale=1 1 1
- link RL_hip_shoulder: geometry collision cylinder length=0.035 radius=0.039; visual cylinder length=0.035 radius=0.039
- link RL_knee: geometry collision box size=0.016 0.016 0.18341; visual mesh filename=package://cyberdog2/meshes/visual/knee.stl scale=1 1 1
- link RR_hip_shoulder: geometry collision cylinder length=0.035 radius=0.039; visual cylinder length=0.035 radius=0.039
- link RR_knee: geometry collision box size=0.016 0.016 0.18341; visual mesh filename=package://cyberdog2/meshes/visual/knee.stl scale=1 1 1
- link body: geometry collision box size=0.4 0.25 0.109; visual mesh filename=package://cyberdog2/meshes/visual/body.stl scale=1 1 1
- link head: geometry 

File: o2/urdf/o2_description.urdf (robot description, URDF)
Before this commit: robot O2with_inertial, 7 links, 6 joints
Links:
- link L1: geometry collision box size=0.03 0.03 0.2; visual box size=0.03 0.03 0.2
- link L2: geometry collision box size=0.03 0.03 0.2; visual box size=0.03 0.03 0.2
- link L3: geometry collision cylinder length=0.02 radius=0.0948; visual cylinder length=0.02 radius=0.0948
- link R1: geometry collision box size=0.03 0.03 0.2; visual box size=0.03 0.03 0.2
- link R2: geometry collision box size=0.03 0.03 0.2; visual box size=0.03 0.03 0.2
- link R3: geometry collision cylinder length=0.02 radius=0.0948; visual cylinder length=0.02 radius=0.0948
- link base: geometry collision box size=0.4 0.2 0.2; visual box size=0.4 0.2 0.2
